File: CM4_GPOI.kicad_sch (KiCad schematic)
At the start: 19 parts, among them J5 61900419521, M2 CM4-GPIO, U11 EMC2301, U5 74LVC1G07SE-7

Commit message: feat: TPM and GPIO (#22)
Parts:
- added C10, C11, C9: 100n, Hardware Components:C_0402_1005Metric, symbol Hardware Components:C_100n_0402_16V
- added C12: 4u7, Hardware Components:C_0402_1005Metric, symbol Hardware Components:C_4u7_0402_16V
- added J4: Conn_02x04_Odd_Even, Hardware Components:Conn_PinHeader_2x05_P2.54mm_Vertical, symbol Hardware Components:Conn_PinHeader_2x05_P2.54mm_Vertical
- added R19, R20: 10k, Hardware Components:R_0402_1005Metric, symbol Hardware Components:R_10k_0402_50V
- added SW1: SW_Push, Hardware Components:SW_Panasonic_EVQPUC, symbol Hardware Components:SW_Panasonic_EVQPUC02K
- added U9: SLB9672XU20FW1612XTMA1, Hardware Components:UQFN-32-1, symbol Hardware Components:SLB9672XU20FW1610XTMA1
- C2: footprint Capacitor_SMD:C_0402_1005Metric -> Hardware Components:C_0402_1005Metric; symbol HomeLabIO:C -> Hardware Components:C_100n_0402_16V
- D1: footprint LED_SMD:LED_0603_1608Metric -> Hardware Components:LED_0603_1608Metric; symbol HomeLabIO:LED -> Hardware Components:LED_G_0603_LTST-C191KGKT
- D2: footprint LED_SMD:LED_0603_1608Metric -> Hardware Components:LED_0603_1608Metric; symbol HomeLabIO:LED -> Hardware Components:LED_R_0603_LTST-C191KRKT
- J5: footprint HomeLabIO:TE_640455-4 -> Hardware Components:Conn_PinHeader_1x04_P2.54mm_Horizontal_Latch; symbol HomeLabIO:640455-4 -> Hardware Components:Conn_PinHeader_1x04_P2.54mm_Horizontal_Latch
- M2: footprint HomeLabIO:HIROSE_DF40C-100DS-0.4V_51_ -> Hardware Components:Conn_Socket_HIROSE_DF40_2x50_DF40C-100DS-0.4V; symbol HomeLabIO:CM4-GPIO -> Hardware Components:Compute-Module-4_GPIO
- Module1: footprint HomeLabIO:Raspberry-Pi-4-Compute-Module -> Hardware Components:Compute-Module-4-H1; symbol HomeLabIO:ComputeModule4-CM4 -> Hardware Components:Compute-Module-4_H1; MPN (none) -> SC0294; Manufacturer Hirose -> Rapberry Pi
- R4, R5: footprint Resistor_SMD:R_0402_1005Metric -> Hardware Components:R_0402_1005Metric; symbol HomeLabIO:R -> Hardware Components:R_1k_0402_75V
- R8: footprint Resistor_SMD:R_0402_1005Metric -> Hardware Components:R_0402_1005Metric; symbol HomeLabIO:R -> Hardware Components:R_36k_0402_50V
- U11: footprint HomeLabIO:MSOP8_MC_MCH -> Hardware Components:MSOP8_MC_MCH; symbol HomeLabIO:EMC2301 -> Hardware Components:Driver_EMC2301
- U5: footprint Package_TO_SOT_SMD:SOT-353_SC-70-5 -> Hardware Components:SOT-353_SC-70-5; symbol HomeLabIO:74LVC1G07SE-7 -> Hardware Components:74LVC1G07SE-7
Connections:
- net +3.3V: now also C10.1, C11.1, C12.1, C9.1, J4.1 (Pin_1), R19.1, R20.1, U9.1 (VDD), U9.14 (VDD), U9.22 (VDD), U9.8 (NCI/VDD)
- net GND: now also C10.2, C11.2, C12.2, C9.2, J4.6 (Pin_6), J4.9 (Pin_9), SW1.2, U9.16 (NCI/GND), U9.2 (GND), U9.23 (GND), U9.32 (GND), U9.33 (GND), U9.9 (GND)
- net TACH: now reaches J5.3 (Pin_3), R8.2, U11.6 (TACH)
- net PWM: now reaches J5.4 (Pin_4), U11.5 (PWM)
- net USER_BTN: now reaches M2.27 (GPIO20)
- net USER_BTN: now also R20.2, SW1.1
- net TPM.CS: now reaches M2.37 (GPIO7)
- net TPM.CS: now also R19.2, U9.20 (CS#)
- net TPM.SCLK: now reaches M2.38 (GPIO11)
- net TPM.SCLK: now also J4.8 (Pin_8), U9.19 (SCLK)
- net GPIO8: now reaches M2.39 (GPIO8)
- net GPIO8: now also J4.10 (Pin_10)
- net TPM.MISO: now reaches M2.40 (GPIO9)
- net TPM.MISO: now also J4.2 (Pin_2), U9.24 (MISO)
- net TPM.MOSI: now reaches M2.44 (GPIO10)
- net TPM.MOSI: now also J4.4 (Pin_4), U9.21 (MOSI)
- net TPM.IRQ: now reaches M2.45 (GPIO24)
- net TPM.IRQ: now also U9.18 (PIRQ#)
- net GPIO4: now reaches M2.54 (GPIO4)
- net GPIO4: now also J4.7 (Pin_7)
- net GPIO3: now reaches M2.56 (GPIO3)
- net GPIO3: now also J4.3 (Pin_3)
- net GPIO2: now reaches M2.58 (GPIO2)
- net GPIO2: now also J4.5 (Pin_5)
- no-connect marks 49 -> 43
Other:
- note added: "TPM 2.0"
- title: (none) -> HomeLabIO
- moved on the sheet: C2, D2, Module1, R5, R8, TP1, U5
